File: apec-gear-pump-board.kicad_sch (KiCad schematic)
At the start: 15 parts, among them J1 Screw_Terminal_01x06, J2 Screw_Terminal_01x02, J4 Screw_Terminal_01x06, U1 74LV1T125, U2 74LV1T125, U3 74LV1T125

Commit message: More silk screen on the back, changed pinout on the connectors, to put optional pins towards one edge
Connections:
- net DIRECTION_3V3: now also J4.6 (Pin_6); no longer J4.4 (Pin_4)
- net DIRECTION_5V: now also J1.6 (DIRECTION); no longer J1.3 (SPEED_IN)
- net GND: now also J1.4 (SIGNAL_GND); no longer J1.6 (DIRECTION)
- net SPEED_IN_3V3: now also J4.4 (Pin_4); no longer J4.6 (Pin_6)
- net SPEED_IN_5V: now also J1.3 (SPEED_IN); no longer J1.5 (TACHO_OUT)
- net TACHO_OUT_5V: now also J1.5 (TACHO_OUT); no longer J1.4 (SIGNAL_GND)
Changed lines of the file:
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@@
     (stroke (width 0) (type default))
+  )
+  (global_label "TACHO_OUT_5V" (shape output) (at 119.38 48.26 180) (fields_autoplaced)
+    (effects (font (size 1.27 1.27)) (justify right))
+    (property "Intersheetrefs" "${INTERSHEET_REFS}" (at 102.5457 48.26 0)
+      (effects (font (size 1.27 1.27)) (justify right) hide)
+    )
   )
   (global_label "DIRECTION_3V3" (shape input) (at 46.99 133.35 180) (fields_autoplaced)
@@
     )
   )
-  (global_label "SPEED_IN_3V3" (shape output) (at 43.18 43.18 0) (fields_autoplaced)
-    (effects (font (size 1.27 1.27)) (justify left))
-    (property "Intersheetrefs" "${INTERSHEET_REFS}" (at 59.5908 43.18 0)
-      (effects (font (size 1.27 1.27)) (justify left) hide)
-    )
-  )
   (global_label "SPEED_IN_5V" (shape output) (at 109.22 93.98 0) (fields_autoplaced)
     (effects (font (size 1.27 1.27)) (justify left))
@@
     )
   )
+  (global_label "SPEED_IN_3V3" (shape output) (at 43.18 48.26 0) (fields_autoplaced)
+    (effects (font (size 1.27 1.27)) (justify left))
+    (property "Intersheetrefs" "${INTERSHEET_REFS}" (at 59.5908 48.26 0)
+      (effects (font (size 1.27 1.27)) (justify left) hide)
+    )
+  )
+  (global_label "DIRECTION_5V" (shape input) (at 119.38 50.8 180) (fields_autoplaced)
+    (effects (font (size 1.27 1.27)) (justify right))
+    (property "Intersheetrefs" "${INTERSHEET_REFS}" (at 103.3319 50.8 0)
+      (effects (font (size 1.27 1.27)) (justify right) hide)
+    )
+  )
   (global_label "DIRECTION_5V" (shape output) (at 91.44 133.35 0) (fields_autoplaced)
     (effects (font (size 1.27 1.27)) (justify left))
@@
     )
   )
-  (global_label "SPEED_IN_5V" (shape input) (at 119.38 48.26 180) (fields_autoplaced)
-    (effects (font (size 1.27 1.27)) (justify right))
-    (property "Intersheetrefs" "${INTERSHEET_REFS}" (at 104.1787 48.26 0)
-      (effects (font (size 1.27 1.27)) (justify right) hide)
-    )
-  )
-  (global_label "DIRECTION_5V" (shape input) (at 119.38 43.18 180) (fields_autoplaced)
-    (effects (font (size 1.27 1.27)) (justify right))
-    (property "Intersheetrefs" "${INTERSHEET_REFS}" (at 103.3319 43.18 0)
-      (effects (font (size 1.27 1.27)) (justify right) hide)
-    )
-  )
-  (global_label "DIRECTION_3V3" (shape output) (at 43.18 48.26 0) (fields_autoplaced)
+  (global_label "DIRECTION_3V3" (shape output) (at 43.18 43.18 0) (fields_autoplaced)
     (effects (font (size 1.27 1.27)) (justify left))
-    (property "Intersheetrefs" "${INTERSHEET_REFS}" (at 60.4376 48.26 0)
+    (property "Intersheetrefs" "${INTERSHEET_REFS}" (at 60.4376 43.18 0)
       (effects (font (size 1.27 1.27)) (justify left) hide)
     )
@@
     )
   )
-  (global_label "TACHO_OUT_5V" (shape output) (at 119.38 45.72 180) (fields_autoplaced)
+  (global_label "SPEED_IN_5V" (shape input) (at 119.38 43.18 180) (fields_autoplaced)
     (effects (font (size 1.27 1.27)) (justify right))
-    (property "Intersheetrefs" "${INTERSHEET_REFS}" (at 102.5457 45.72 0)
+    (property "Intersheetrefs" "${INTERSHEET_REFS}" (at 104.1787 43.18 0)
       (effects (font (size 1.27 1.27)) (justify right) hide)
     )
@@
     )
   )
+  (symbol (lib_id "power:GND") (at 119.38 45.72 270) (unit 1)
+    (in_bom yes) (on_board yes) (dnp no) (fields_autoplaced)
+    (property "Reference" "#PWR04" (at 113.03 45.72 0)
+      (effects (font (size 1.27 1.27)) hide)
+    )
+    (property "Value" "GND" (at 115.57 45.72 90)
+      (effects (font (size 1.27 1.27)) (justify right))
+    )
+    (property "Footprint" "" (at 119.38 45.72 0)
+      (effects (font (size 1.27 1.27)) hide)
+    )
+    (property "Datasheet" "" (at 119.38 45.72 0)
+      (effects (font (size 1.27 1.27)) hide)
+    )
+    (pin "1")
+    (instances
+      (project "apec-gear-pump-board"
+        (path "/f01ed30c-0f0a-4868-bb0f-e4c4d93b4399"
+          (reference "#PWR04") (unit 1)
+        )
+      )
+    )
+  )
   (symbol (lib_id "Device:C_Small") (at 78.74 59.69 90) (unit 1)
     (in_bom yes) (on_board yes) (dnp no) (fields_autoplaced)
@@
         )
       )
-    )
-  )
-  (symbol (lib_id "power:GND") (at 119.38 50.8 270) (unit 1)
-    (in_bom yes) (on_board yes) (dnp no) (fields_autoplaced)
-    (property "Reference" "#PWR04" (at 113.03 50.8 0)
-      (effects (font (size 1.27 1.27)) hide)
-    )
-    (property "Value" "GND" (at 115.57 50.8 90)
-      (effects (font (size 1.27 1.27)) (justify right))
-    )
-    (property "Footprint" "" (at 119.38 50.8 0)
-      (effects (font (size 1.27 1.27)) hide)
-    )
-    (property "Datasheet" "" (at 119.38 50.8 0)
-      (effects (font (size 1.27 1.27)) hide)
-    )
-    (pin "1")
-    (instances
-      (project "apec-gear-pump-board"
-        (path "/f01ed30c-0f0a-4868-bb0f-e4c4d93b4399"
-          (reference "#PWR04") (unit 1)
-        )
-      )
